Commit message: Initial commit: AMR project with LiDAR, ESP32, and EKF configuration

File: src/my_robot_description/urdf/amr_robot.SLDASM.urdf (robot description, URDF)
Before this commit: robot my_amr_robot, 14 links, 13 joints
Links:
- link Tof_BL_link: geometry collision mesh filename=package:/my_robot_description/mesh/Tof_BL_link.STL; visual mesh filename=package:/my_robot_description/mesh/Tof_BL_link.STL
- link Tof_BR_link: geometry collision mesh filename=package:/my_robot_description/mesh/Tof_BR_link.STL; visual mesh filename=package:/my_robot_description/mesh/Tof_BR_link.STL
- link Tof_FL_link: geometry collision mesh filename=package:/my_robot_description/mesh/Tof_FL_link.STL; visual mesh filename=package:/my_robot_description/mesh/Tof_FL_link.STL
- link Tof_FR_link: geometry collision mesh filename=package:/my_robot_description/mesh/Tof_FR_link.STL; visual mesh filename=package:/my_robot_description/mesh/Tof_FR_link.STL
- link Tof_F_Link: geometry collision mesh filename=package:/my_robot_description/mesh/Tof_F_Link.STL; visual mesh filename=package:/my_robot_description/mesh/Tof_F_Link.STL
- link back_left_wheel_link: geometry collision cylinder length=0.07 radius=0.08; visual mesh filename=package:/my_robot_description/mesh/back_left_wheel_link.STL
- link back_right_wheel_link: geometry collision cylinder length=0.07 radius=0.08; visual mesh filename=package:/my_robot_description/mesh/back_right_wheel_link.STL
- link base_link: geometry collision mesh filename=package:/my_robot_description/mesh/base_link.STL; visual mesh filename=package:/my_robot_description/mesh/base_link.STL
- link camera_link: geometry collision mesh filename=package:/my_robot_description/mesh/camera_link.STL; visual mesh filename=package:/my_robot_description/mesh/camera_link.STL
- link front_left_wheel_link: geometry collision cylinder length=0.07 radius=0.08; visual mesh filename=package:/my_robot_description/mesh/front_left_wheel_link.STL
- link front_right_wheel_link: geometry collision cylinder length=0.07 radius=0.08; visual mesh filename=package:/my_robot_description/mesh/front_right_wheel_link.S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
- link gps_link: geometry collision mesh filename=package:/my_robot_description/mesh/gps_link.STL; visual mesh filename=package:/my_robot_description/mesh/gps_link.STL
- link lidar_link: geometry collision mesh filename=package:/my_robot_description/mesh/lidar_link.STL; visual mesh filename=package:/my_robot_description/mesh/lidar_link.STL
